File: ETH_PHY.sch (KiCad schematic (older format))
At the start: 0 parts

Commit message: update for RTL8211D,
Parts:
- added C? (x3): C475,0603, Capacitor_SMD:C_0603_1608Metric_Pad1.05x0.95mm_HandSolder, symbol taobao-c:C475,0603
- added C? (x3): C12pf,0603, symbol Device:C_Small
- added R? (x3): R203,0603, Resistor_SMD:R_0603_1608Metric_Pad1.05x0.95mm_HandSolder, symbol taobao-r:R203,0603
- added R? (x3): R0,0603, Resistor_SMD:R_0603_1608Metric_Pad1.05x0.95mm_HandSolder, symbol taobao-r:R0,0603
- added R? (x2): R433,0603, Resistor_SMD:R_0603_1608Metric_Pad1.05x0.95mm_HandSolder, symbol taobao-r:R433,0603
- added R?: R563,0603, Resistor_SMD:R_0603_1608Metric_Pad1.05x0.95mm_HandSolder, symbol taobao-r:R563,0603
- added U?: RTL8211D,RTL8211E, symbol taobao-components:RTL8211D,RTL8211E
- added U? (x3): AP2127K-ADJTRG1, symbol taobao-components:AP2127K-ADJTRG1
Connections:
- new net: R?.2, R?.2, U?.4 (ADJ) (x3)
- new net CLK125: R?.1
- new net GCLKIN: C?.2, R?.2
- new net GMAC-2V5: C?.1, R?.1, U?.5 (VOUT)
- new net GMAC-3V: C?.1, R?.1, U?.5 (VOUT)
- new net GMAC-PWR-EN: U?.3 (EN), U?.3 (EN)
- new net GND: C?.1, C?.1, C?.1, C?.2, C?.2, C?.2, R?.1, R?.1, R?.1, U?.2 (GND), U?.2 (GND), U?.2 (GND)
- new net GRXCK: C?.2, R?.2
- new net GTXCK: C?.2, R?.2
- new net RXCLK: R?.1
- new net TXCLK: R?.1
- new net V_IO: U?.1 (INPUT), U?.1 (INPUT), U?.1 (INPUT), U?.3 (EN)
- new net V_PD: C?.1, R?.1, U?.5 (VOUT)

Commit message: update for EPHY,
Parts:
- removed U?: RTL8211D,RTL8211E, symbol taobao-components:RTL8211D,RTL8211E
- added C? (x2): C27pf,0603, Capacitor_SMD:C_0603_1608Metric_Pad1.05x0.95mm_HandSolder, symbol taobao-c:C27pf,0603
- added R?: 2K49,0603, symbol Device:R_Small
- added U?: RTL8211D,RTL8211E, symbol taobao-components:RTL8211D,RTL8211E
- added Y?: O_25M,3225, Oscillator:Oscillator_SMD_Abracon_ASE-4Pin_3.2x2.5mm_HandSoldering, symbol taobao-osc:O_25M,3225
Connections:
- net GND: now also C?.2, C?.2, R?.1, U?.47 (GND), U?.49 (PAD), Y?.2
- new net: C?.1, U?.42 (CKXTAL1), Y?.1
- new net: C?.1, U?.43 (CKXTAL2), Y?.3
- new net AVDD10: U?.3 (AVDD10), U?.9 (AVDD10)
- new net DVDD10: U?.28 (DVDD10), U?.36 (DVDD10)
- new net EPHY-AVDD33: U?.6 (AVDD33)
- new net LED0-AD0: U?.34 (PHY_AD[0]/LED0)
- new net LED1-AD1: U?.35 (PHY_AD[1]/LED1)
- new net LED2-RXDLY: U?.32 (RXDLY/LED2)
- new net MDC: U?.30 (MDC)
- new net MDI0+: U?.1 (MDIP0)
- new net MDI0-: U?.2 (MDIN0)
- new net MDI1+: U?.4 (MDIP1)
- new net MDI1-: U?.5 (MDIN1)
- new net MDI2+: U?.7 (MDIP2)
- new net MDI2-: U?.8 (MDIN2)
- new net MDI3+: U?.10 (MDIP3)
- new net MDI3-: U?.11 (MDIN3)
- new net MDIO: U?.31 (MDIO)
- new net PHYRSTB: U?.29 (PHYRSTB)
- new net PMEB: U?.33 (PME)
- new net REGOUT: U?.48 (REG_OUT)
- new net RSET: R?.2, U?.39 (RSET)
- new net TXCTL: U?.27 (TXCTL)
- new net TXD2: U?.25 (TXD2)
- new net TXD3: U?.26 (TXD3)

Commit message: update for EPHY,
Connections:
- net RXCLK: now also U?.19 (RXC)
- net TXCLK: now also U?.22 (GTX_CLK)
- net RXCTL-AD2: now reaches U?.13 (RXCTL)
- net RXD0-SELRGV: now reaches U?.14 (RXD0/SELRGV)
- net EPHY-VDD25: now reaches U?.15 (DVDD33)
- net EPHY-VDD25: now also U?.21 (DVDD33)
- net RXD1-TXDLY: now reaches U?.16 (RXD1/TXDLY)
- net RXD2-AN0: now reaches U?.17 (RXD2/AN[0])
- net RXD3-AN1: now reaches U?.18 (RXD3/AN[1])
- net INTB: now reaches U?.20 (INT)
- net TXD0: now reaches U?.23 (TXD0)
- net TXD1: now reaches U?.24 (TXD1)
Changed lines of the file:
@@
 Wire Wire Line
 	7700 4300 8750 4300
+Text Label 9350 5750 1    50   ~ 0
+RXCTL-AD2
+Text Label 9450 5750 1    50   ~ 0
+RXD0-SELRGV
+Text Label 9550 5750 1    50   ~ 0
+EPHY-VDD25
+Text Label 9650 5750 1    50   ~ 0
+RXD1-TXDLY
+Text Label 9750 5750 1    50   ~ 0
+RXD2-AN0
+Text Label 9850 5750 1    50   ~ 0
+RXD3-AN1
+Text Label 9950 5750 1    50   ~ 0
+RXCLK
+Text Label 10050 5750 1    50   ~ 0
+INTB
+Text Label 10150 5750 1    50   ~ 0
+EPHY-VDD25
+Text Label 10250 5750 1    50   ~ 0
+TXCLK
+Text Label 10350 5750 1    50   ~ 0
+TXD0
+Text Label 10450 5750 1    50   ~ 0
+TXD1
+Wire Wire Line
+	9350 5000 9350 5750
+Wire Wire Line
+	9450 5000 9450 5750
+Wire Wire Line
+	9550 5000 9550 5750
+Wire Wire Line
+	9650 5000 9650 5750
+Wire Wire Line
+	9750 5000 9750 5750
+Wire Wire Line
+	9850 5000 9850 5750
+Wire Wire Line
+	9950 5000 9950 5750
+Wire Wire Line
+	10050 5000 10050 5750
+Wire Wire Line
+	10150 5000 10150 5750
+Wire Wire Line
+	10250 5000 10250 5750
+Wire Wire Line
+	10350 5000 10350 5750
+Wire Wire Line
+	10450 5000 10450 5750
 $EndSCHEMATC

Commit message: update for EPHY,
Parts:
- added C? (x13): C104,0603, Capacitor_SMD:C_0603_1608Metric_Pad1.05x0.95mm_HandSolder, symbol taobao-c:C104,0603
- added C? (x2): C226,6.3v,0603, Capacitor_SMD:C_0603_1608Metric_Pad1.05x0.95mm_HandSolder, symbol taobao-c:C226,6.3v,0603
- added C? (x3): C102,0603, Capacitor_SMD:C_0603_1608Metric_Pad1.05x0.95mm_HandSolder, symbol taobao-c:C102,0603
- added L?: L_4.7uH,CD43, w_smd_inductors:inductor_smd_4.8x2.8mm, symbol taobao-l:L_4.7uH,CD43
- added R? (x15): R472,0603, Resistor_SMD:R_0603_1608Metric_Pad1.05x0.95mm_HandSolder, symbol taobao-r:R472,0603
- added R? (x2): R751,0603, Resistor_SMD:R_0603_1608Metric_Pad1.05x0.95mm_HandSolder, symbol taobao-r:R751,0603
- added R? (x2): R0,0603, Resistor_SMD:R_0603_1608Metric_Pad1.05x0.95mm_HandSolder, symbol taobao-r:R0,0603
- added R?: R152,0603, Resistor_SMD:R_0603_1608Metric_Pad1.05x0.95mm_HandSolder, symbol taobao-r:R152,0603
- added R? (x2): R473,0603, Resistor_SMD:R_0603_1608Metric_Pad1.05x0.95mm_HandSolder, symbol taobao-r:R473,0603
- added R?: R514,0603, Resistor_SMD:R_0603_1608Metric_Pad1.05x0.95mm_HandSolder, symbol taobao-r:R514,0603
- added U?: HANRUN_HR911130C, symbol taobao-components:HANRUN_HR911130C
Connections:
- net EPHY-AVDD33 is gone; now on net GMAC-3V: U?.6 (AVDD33)
- net EPHY-VDD25 is gone; now on net GMAC-2V5: U?.15 (DVDD33), U?.21 (DVDD33)
- net AVDD10: now also C?.1, C?.1, C?.1, C?.1, L?.2, R?.2
- net DVDD10: now also C?.1, C?.1, R?.1
- net GMAC-2V5: now also C?.1, C?.1, R?.1, R?.1, R?.1, R?.1, R?.1, R?.1
- net GMAC-3V: now also C?.1, C?.1, C?.1, C?.1, C?.1, R?.1, R?.1, R?.1, R?.2, U?.14 (LED_ACT_P)
- net GND: now also C?.1, C?.1, C?.2, C?.2, C?.2, C?.2, C?.2, C?.2, C?.2, C?.2, C?.2, C?.2, C?.2, C?.2, C?.2, C?.2, C?.2, C?.2, C?.2, R?.2, R?.2, R?.2, R?.2, R?.2, R?.2, R?.2, R?.2, U?.12 (LED_LINK_N), U?.15 (SHIELD), U?.16 (SHIELD)
- net INTB: now also R?.2
- net LED0-AD0: now also R?.1, R?.2
- net LED1-AD1: now also R?.1, R?.1, R?.2
- net LED2-RXDLY: now also R?.1, R?.2
- net MDI0+: now also U?.2 (MDI0+)
- net MDI0-: now also U?.3 (MDI0-)
- net MDI1+: now also U?.4 (MDI1+)
- net MDI1-: now also U?.7 (MDI1-)
- net MDI2+: now also U?.5 (MDI2+)
- net MDI2-: now also U?.6 (MDI2-)
- net MDI3+: now also U?.8 (MDI3+)
- net MDI3-: now also U?.9 (MDI3-)
- net PHYRSTB: now also C?.2, R?.1
- net PMEB: now also R?.2
- net REGOUT: now also L?.1
- net RXCTL-AD2: now also R?.1
- net RXD0-SELRGV: now also R?.1, R?.2
- net RXD1-TXDLY: now also R?.1, R?.2
- net RXD2-AN0: now also R?.1, R?.2
- net RXD3-AN1: now also R?.1, R?.2
- net MDIO renamed EMDIO
- net EMDIO: now also R?.2
- new net COMMON_CT: C?.1, R?.2, U?.1 (COMMON_CT)
- new net EPHY-DVD33: R?.1, R?.1
- new net LED-AD0: R?.1
- new net LED_ACT_P: C?.1, R?.2, U?.13 (LED_ACT_N)
- new net LED_LINK_P: C?.1, R?.2, U?.11 (LED_LINK_P)
Other:
- moved on the sheet: C?, R?, U?
