File: USB.sch (KiCad schematic (older format))
At the start: 0 parts

Commit message: add USB HOST,
Parts:
- added C? (x2): C104,0603, Capacitor_SMD:C_0603_1608Metric_Pad1.05x0.95mm_HandSolder, symbol taobao-c:C104,0603
- added C?: CP100uf,10V, Capacitor_SMD:CP_Elec_6.3x5.3, symbol taobao-cp:CP100uf,10V
- added C?: C475,0603, Capacitor_SMD:C_0603_1608Metric_Pad1.05x0.95mm_HandSolder, symbol taobao-c:C475,0603
- added C?: CP22uf,16V, Capacitor_SMD:CP_Elec_4x5.3, symbol taobao-cp:CP22uf,16V
- added FB?: Ferrite_Bead_Small, symbol Device:Ferrite_Bead_Small
- added J?: USB_B_Micro, symbol Connector:USB_B_Micro
- added J?: Conn_01x02, symbol Connector_Generic:Conn_01x02
- added Q?: AO3423, symbol taobao-components:AO3423
- added Q?: 2N3904(1AM), Package_TO_SOT_THT:TO-92_Inline, symbol taobao-transistor:2N3904(1AM)
- added R? (x2): R103,0603, Resistor_SMD:R_0603_1608Metric_Pad1.05x0.95mm_HandSolder, symbol taobao-r:R103,0603
- added R? (x2): R0,0603, Resistor_SMD:R_0603_1608Metric_Pad1.05x0.95mm_HandSolder, symbol taobao-r:R0,0603
- added R?: R_NC,0805, Resistor_SMD:R_0805_2012Metric_Pad1.15x1.40mm_HandSolder, symbol taobao-components:R_NC,0805
- added R? (x2): R202,0603, Resistor_SMD:R_0603_1608Metric_Pad1.05x0.95mm_HandSolder, symbol taobao-r:R202,0603
- added R?: R104,0603, Resistor_SMD:R_0603_1608Metric_Pad1.05x0.95mm_HandSolder, symbol taobao-r:R104,0603
- added R?: R102,0603, Resistor_SMD:R_0603_1608Metric_Pad1.05x0.95mm_HandSolder, symbol taobao-r:R102,0603
- added R?: R_NC,0603, Resistor_SMD:R_0603_1608Metric_Pad1.05x0.95mm_HandSolder, symbol taobao-components:R_NC,0603
- added R?: R472,0603, Resistor_SMD:R_0603_1608Metric_Pad1.05x0.95mm_HandSolder, symbol taobao-r:R472,0603
- added U? (x3): ACM2012, symbol taobao-components:ACM2012
- added U?: SY6280AAC, symbol taobao-components:SY6280AAC
- added U?: DUAL_USB-A-VERTICAL, symbol taobao-components:DUAL_USB-A-VERTICAL
Connections:
- new net: FB?.2, J?.1 (VBUS)
- new net: J?.2 (D-), U?.2
- new net: J?.3 (D+), U?.1
- new net: J?.4 (ID), R?.1, R?.2
- new net: R?.2, U?.3
- new net: R?.2, U?.4
- new net: C?.2, Q?.1 (G), Q?.3 (C), R?.2
- new net: Q?.1 (B), R?.1
- new net: R?.1, U?.3 (FALG)
- new net: R?.1, R?.2, U?.4 (EN)
- new net: U?.4, U?.A2 (D1-)
- new net: U?.3, U?.A3 (D1+)
- new net: U?.4, U?.B2 (D2-)
- new net: U?.3, U?.B3 (D2+)
- new net GND: C?.2, C?.2, C?.2, C?.2, J?.5 (GND), J?.6 (Shield), Q?.2 (E), R?.2, R?.2, U?.2 (GND), U?.3 (SHIELD3), U?.4 (SHIELD4), U?.A4 (GND1), U?.B4 (GND2)
- new net HOST-VBUS: C?.1, C?.1, R?.1, U?.1 (VOUT1), U?.A1 (VBUS1), U?.B1 (VBUS2)
- new net USB-DN: R?.1
- new net USB-DN1: U?.1
- new net USB-DN2: U?.1
- new net USB-DN3: J?.2 (Pin_2)
- new net USB-DP: R?.1
- new net USB-DP1: U?.2
- new net USB-DP2: U?.2
- new net USB-DP3: J?.1 (Pin_1)
- new net USB-ID: R?.1
- new net USB0-DRVVBUS: R?.2, R?.2
- new net USBVBUS: C?.1, C?.1, FB?.1, Q?.3 (D)
- new net Vcc-5V: C?.1, Q?.2 (S), R?.1, R?.2, U?.5 (IN)
- new net Vcc-io: R?.2
- new net Vio: R?.1, R?.1

Commit message: update,
Parts:
- removed C? (x2): C104,0603, Capacitor_SMD:C_0603_1608Metric_Pad1.05x0.95mm_HandSolder, symbol taobao-c:C104,0603
- removed C?: CP100uf,10V, Capacitor_SMD:CP_Elec_6.3x5.3, symbol taobao-cp:CP100uf,10V
- removed C?: C475,0603, Capacitor_SMD:C_0603_1608Metric_Pad1.05x0.95mm_HandSolder, symbol taobao-c:C475,0603
- removed C?: CP22uf,16V, Capacitor_SMD:CP_Elec_4x5.3, symbol taobao-cp:CP22uf,16V
- removed FB?: Ferrite_Bead_Small, symbol Device:Ferrite_Bead_Small
- removed J?: USB_B_Micro, symbol Connector:USB_B_Micro
- removed J?: Conn_01x02, symbol Connector_Generic:Conn_01x02
- removed Q?: AO3423, symbol taobao-components:AO3423
- removed Q?: 2N3904(1AM), Package_TO_SOT_THT:TO-92_Inline, symbol taobao-transistor:2N3904(1AM)
- removed R? (x2): R103,0603, Resistor_SMD:R_0603_1608Metric_Pad1.05x0.95mm_HandSolder, symbol taobao-r:R103,0603
- removed R? (x2): R0,0603, Resistor_SMD:R_0603_1608Metric_Pad1.05x0.95mm_HandSolder, symbol taobao-r:R0,0603
- removed R?: R_NC,0805, Resistor_SMD:R_0805_2012Metric_Pad1.15x1.40mm_HandSolder, symbol taobao-components:R_NC,0805
- removed R? (x2): R202,0603, Resistor_SMD:R_0603_1608Metric_Pad1.05x0.95mm_HandSolder, symbol taobao-r:R202,0603
- removed R?: R104,0603, Resistor_SMD:R_0603_1608Metric_Pad1.05x0.95mm_HandSolder, symbol taobao-r:R104,0603
- removed R?: R102,0603, Resistor_SMD:R_0603_1608Metric_Pad1.05x0.95mm_HandSolder, symbol taobao-r:R102,0603
- removed R?: R_NC,0603, Resistor_SMD:R_0603_1608Metric_Pad1.05x0.95mm_HandSolder, symbol taobao-components:R_NC,0603
- removed R?: R472,0603, Resistor_SMD:R_0603_1608Metric_Pad1.05x0.95mm_HandSolder, symbol taobao-r:R472,0603
- removed U? (x3): ACM2012, symbol taobao-components:ACM2012
- removed U?: SY6280AAC, symbol taobao-components:SY6280AAC
- removed U?: DUAL_USB-A-VERTICAL, symbol taobao-components:DUAL_USB-A-VERTICAL
- added C?: C104,0603, Capacitor_SMD:C_0603_1608Metric_Pad1.05x0.95mm_HandSolder, symbol taobao-c:C104,0603
- added J?: USB_B_Micro, symbol Connector:USB_B_Micro
- added R?: R103,0603, Resistor_SMD:R_0603_1608Metric_Pad1.05x0.95mm_HandSolder, symbol taobao-r:R103,0603
Connections:
- net GND: now also C?.2, J?.4 (ID), J?.5 (GND), J?.6 (Shield), R?.2
- net USB-DN1: now also J?.3 (D+)
- net USBVBUS: now also C?.1, J?.1 (VBUS)
- net Vcc-io: now also R?.1
- new net USB-DN0: J?.2 (D-)
