File: USB.sch (KiCad schematic (older format))
At the start: 3 parts

Commit message: update power mark,
Connections:
- net labels added: VCC-5V, VCC-IO
- net labels removed: Vcc-5V, Vcc-io
Changed lines of the file:
@@
 $Descr A3 16535 11693
 encoding utf-8
-Sheet 5 33
+Sheet 5 34
 Title ""
 Date ""
@@
 $EndComp
 $Comp
-L taobao-components:Vcc-io #PWR?
-U 1 1 5C2327E9
-P 7350 4700
-F 0 "#PWR?" H 7350 4550 50  0001 C CNN
-F 1 "Vcc-io" H 7400 4850 50  0000 C CNN
-F 2 "" H 7350 4700 50  0001 C CNN
-F 3 "" H 7350 4700 50  0001 C CNN
-	1    7350 4700
-	1    0    0    -1
-$EndComp
-$Comp
 L taobao-r:R103,0603 R?
 U 1 1 5C232926
@@
 F 3 "" H 8650 5100 50  0001 C CNN
 	1    8650 5100
-	1    0    0    -1
-$EndComp
-$Comp
-L taobao-components:Vcc-5V #PWR?
-U 1 1 5C232B2D
-P 9350 5100
-F 0 "#PWR?" H 9350 4950 50  0001 C CNN
-F 1 "Vcc-5V" H 9400 5250 50  0000 C CNN
-F 2 "" H 9350 5100 50  0001 C CNN
-F 3 "" H 9350 5100 50  0001 C CNN
-	1    9350 5100
 	1    0    0    -1
 $EndComp
@@
 Text Label 9350 5750 2    50   ~ 0
 USB0-ID
+$Comp
+L taobao-components:VCC-IO #PWR?
+U 1 1 5C7D75C3
+P 7350 4700
+F 0 "#PWR?" H 7350 4550 50  0001 C CNN
+F 1 "VCC-IO" H 7400 4850 50  0000 C CNN
+F 2 "" H 7350 4700 50  0001 C CNN
+F 3 "" H 7350 4700 50  0001 C CNN
+	1    7350 4700
+	1    0    0    -1
+$EndComp
+$Comp
+L taobao-components:VCC-5V #PWR?
+U 1 1 5C7DB88A
+P 9350 5100
+F 0 "#PWR?" H 9350 4950 50  0001 C CNN
+F 1 "VCC-5V" H 9400 5250 50  0000 C CNN
+F 2 "" H 9350 5100 50  0001 C CNN
+F 3 "" H 9350 5100 50  0001 C CNN
+	1    9350 5100
+	1    0    0    -1
+$EndComp
 $EndSCHEMATC

Commit message: update for USB,
Parts:
- added C?: C475,0603, Capacitor_SMD:C_0603_1608Metric_Pad1.05x0.95mm_HandSolder, symbol taobao-c:C475,0603
- added Q?: AO3423, symbol taobao-components:AO3423
- added Q?: 2N3904(1AM), Package_TO_SOT_THT:TO-92_Inline, symbol taobao-transistor:2N3904(1AM)
- added R?: R104,0603, Resistor_SMD:R_0603_1608Metric_Pad1.05x0.95mm_HandSolder, symbol taobao-r:R104,0603
- added R?: R202,0603, Resistor_SMD:R_0603_1608Metric_Pad1.05x0.95mm_HandSolder, symbol taobao-r:R202,0603
- added R?: R_NC,0603, Resistor_SMD:R_0603_1608Metric_Pad1.05x0.95mm_HandSolder, symbol taobao-components:R_NC,0603
- added R?: R102,0603, Resistor_SMD:R_0603_1608Metric_Pad1.05x0.95mm_HandSolder, symbol taobao-r:R102,0603
Connections:
- net labels added: USB-DN, USB-DP, USB0-DRVVBUS
- net labels removed: USB-DN0, USB-DN1
- wire segments 20 -> 41
Other:
- moved on the sheet: C?, J?, R?
