File: eMMC.sch (KiCad schematic (older format))
At the start: 26 parts

Commit message: update,
Parts:
- removed C? (x2): C104,0603, Capacitor_SMD:C_0603_1608Metric_Pad1.05x0.95mm_HandSolder, symbol taobao-c:C104,0603
- removed C?: CP100uf,10V, Capacitor_SMD:CP_Elec_6.3x5.3, symbol taobao-cp:CP100uf,10V
- removed C?: C475,0603, Capacitor_SMD:C_0603_1608Metric_Pad1.05x0.95mm_HandSolder, symbol taobao-c:C475,0603
- removed C?: CP22uf,16V, Capacitor_SMD:CP_Elec_4x5.3, symbol taobao-cp:CP22uf,16V
- removed FB?: Ferrite_Bead_Small, symbol Device:Ferrite_Bead_Small
- removed J?: USB_B_Micro, symbol Connector:USB_B_Micro
- removed J?: Conn_01x02, symbol Connector_Generic:Conn_01x02
- removed Q?: AO3423, symbol taobao-components:AO3423
- removed Q?: 2N3904(1AM), Package_TO_SOT_THT:TO-92_Inline, symbol taobao-transistor:2N3904(1AM)
- removed R? (x2): R103,0603, Resistor_SMD:R_0603_1608Metric_Pad1.05x0.95mm_HandSolder, symbol taobao-r:R103,0603
- removed R? (x2): R0,0603, Resistor_SMD:R_0603_1608Metric_Pad1.05x0.95mm_HandSolder, symbol taobao-r:R0,0603
- removed R?: R_NC,0805, Resistor_SMD:R_0805_2012Metric_Pad1.15x1.40mm_HandSolder, symbol taobao-components:R_NC,0805
- removed R? (x2): R202,0603, Resistor_SMD:R_0603_1608Metric_Pad1.05x0.95mm_HandSolder, symbol taobao-r:R202,0603
- removed R?: R104,0603, Resistor_SMD:R_0603_1608Metric_Pad1.05x0.95mm_HandSolder, symbol taobao-r:R104,0603
- removed R?: R102,0603, Resistor_SMD:R_0603_1608Metric_Pad1.05x0.95mm_HandSolder, symbol taobao-r:R102,0603
- removed R?: R_NC,0603, Resistor_SMD:R_0603_1608Metric_Pad1.05x0.95mm_HandSolder, symbol taobao-components:R_NC,0603
- removed R?: R472,0603, Resistor_SMD:R_0603_1608Metric_Pad1.05x0.95mm_HandSolder, symbol taobao-r:R472,0603
- removed U? (x3): ACM2012, symbol taobao-components:ACM2012
- removed U?: SY6280AAC, symbol taobao-components:SY6280AAC
- removed U?: DUAL_USB-A-VERTICAL, symbol taobao-components:DUAL_USB-A-VERTICAL
- added C? (x2): C105,0603, Capacitor_SMD:C_0603_1608Metric_Pad1.05x0.95mm_HandSolder, symbol taobao-c:C105,0603
- added C? (x2): C104,0603, Capacitor_SMD:C_0603_1608Metric_Pad1.05x0.95mm_HandSolder, symbol taobao-c:C104,0603
- added R? (x2): R_NC,0603, Resistor_SMD:R_0603_1608Metric_Pad1.05x0.95mm_HandSolder, symbol taobao-components:R_NC,0603
- added R?: R103,0603, Resistor_SMD:R_0603_1608Metric_Pad1.05x0.95mm_HandSolder, symbol taobao-r:R103,0603
- added U?: EMMC_BGA169, symbol taobao-components:EMMC_BGA169
Connections:
- net GND: now also C?.2, C?.2, C?.2, C?.2, R?.2, R?.2, U?.AA4 (VSSQ), U?.AA6 (VSSQ), U?.K4 (VSSQ), U?.M7 (VSS), U?.P5 (VSS), U?.R10 (VSS), U?.U8 (VSS), U?.Y2 (VSSQ), U?.Y5 (VSSQ)
- new net: R?.1, U?.H6 (RFU/VSS5)
- new net: C?.1, C?.1, U?.K2 (VDDi)
- new net: R?.1, U?.T5 (RFU/VSS4)
- new net V-flash: C?.1, C?.1, R?.2, U?.AA3 (VCCQ), U?.AAS (VCCQ), U?.K6 (VCCQ), U?.M6 (VCC), U?.N5 (VCC), U?.T10 (VCC), U?.U9 (VCC), U?.W4 (VCCQ), U?.Y4 (VCCQ)
- new net eMMC-CLK: U?.W6 (CLK)
- new net eMMC-CMD: R?.1, U?.W5 (CMD)
- new net eMMC-D0: U?.H3 (DATO)
- new net eMMC-D1: U?.H4 (DAT1)
- new net eMMC-D2: U?.H5 (DAT2)
- new net eMMC-D3: U?.J2 (DAT3)
- new net eMMC-D4: U?.J3 (DAT4)
- new net eMMC-D5: U?.J4 (DATS)
- new net eMMC-D6: U?.J5 (DAT6)
- new net eMMC-D7: U?.J6 (DAT7)
- new net eMMC-RST: U?.U5 (RST_n)

Commit message: update,
Parts:
- added R?: R0,0603, Resistor_SMD:R_0603_1608Metric_Pad1.05x0.95mm_HandSolder, symbol taobao-r:R0,0603
Connections:
- net V-flash: now also R?.1
- new net Vcc-io: R?.2
Changed lines of the file:
@@
 $Descr A3 16535 11693
 encoding utf-8
-Sheet 13 14
+Sheet 13 15
 Title ""
 Date ""
@@
 Wire Wire Line
 	13700 5850 12750 5850
+$Comp
+L taobao-components:V-flash #PWR?
+U 1 1 5C5BE76C
+P 5650 2100
+F 0 "#PWR?" H 5650 1950 50  0001 C CNN
+F 1 "V-flash" H 5700 2250 50  0000 C CNN
+F 2 "" H 5650 2100 50  0001 C CNN
+F 3 "" H 5650 2100 50  0001 C CNN
+	1    5650 2100
+	1    0    0    -1
+$EndComp
+$Comp
+L taobao-components:Vcc-io #PWR?
+U 1 1 5C5BE824
+P 4650 2100
+F 0 "#PWR?" H 4650 1950 50  0001 C CNN
+F 1 "Vcc-io" H 4700 2250 50  0000 C CNN
+F 2 "" H 4650 2100 50  0001 C CNN
+F 3 "" H 4650 2100 50  0001 C CNN
+	1    4650 2100
+	1    0    0    -1
+$EndComp
+$Comp
+L taobao-r:R0,0603 R?
+U 1 1 5C5C07D8
+P 5100 2200
+F 0 "R?" V 4850 2200 50  0000 C CNN
+F 1 "R0,0603" V 4950 2200 50  0000 C CNN
+F 2 "Resistor_SMD:R_0603_1608Metric_Pad1.05x0.95mm_HandSolder" H 5100 2200 50  0001 C CNN
+F 3 "~" H 5100 2200 50  0001 C CNN
+	1    5100 2200
+	0    1    1    0
+$EndComp
+Wire Wire Line
+	5000 2200 4650 2200
+Wire Wire Line
+	4650 2200 4650 2100
+Wire Wire Line
+	5200 2200 5650 2200
+Wire Wire Line
+	5650 2200 5650 2100
 $EndSCHEMATC
