File: eMMC.sch (KiCad schematic (older format))
At the start: 9 parts

Commit message: update power mark,
Connections:
- net labels added: VCC-IO
- net labels removed: Vcc-io
Changed lines of the file:
@@
 $Descr A3 16535 11693
 encoding utf-8
-Sheet 13 33
+Sheet 13 34
 Title ""
 Date ""
@@
 $EndComp
 $Comp
-L taobao-components:Vcc-io #PWR?
-U 1 1 5C5BE824
-P 4650 2100
-F 0 "#PWR?" H 4650 1950 50  0001 C CNN
-F 1 "Vcc-io" H 4700 2250 50  0000 C CNN
-F 2 "" H 4650 2100 50  0001 C CNN
-F 3 "" H 4650 2100 50  0001 C CNN
-	1    4650 2100
-	1    0    0    -1
-$EndComp
-$Comp
 L taobao-r:R0,0603 R?
 U 1 1 5C5C07D8
@@
 Wire Wire Line
 	5650 2200 5650 2100
+$Comp
+L taobao-components:VCC-IO #PWR?
+U 1 1 5C7D87CA
+P 4650 2100
+F 0 "#PWR?" H 4650 1950 50  0001 C CNN
+F 1 "VCC-IO" H 4700 2250 50  0000 C CNN
+F 2 "" H 4650 2100 50  0001 C CNN
+F 3 "" H 4650 2100 50  0001 C CNN
+	1    4650 2100
+	1    0    0    -1
+$EndComp
 $EndSCHEMATC

Commit message: update for VCC-FLASH,
Connections:
- net V-flash renamed VCC-FLASH
Changed lines of the file:
@@
-	1    0    0    -1
-$EndComp
-$Comp
-L taobao-components:V-flash #PWR?
-U 1 1 5C256840
-P 12400 2050
-F 0 "#PWR?" H 12400 1900 50  0001 C CNN
-F 1 "V-flash" H 12450 2200 50  0000 C CNN
-F 2 "" H 12400 2050 50  0001 C CNN
-F 3 "" H 12400 2050 50  0001 C CNN
-	1    12400 2050
 	1    0    0    -1
 $EndComp
@@
 Connection ~ 10450 4500
 $Comp
-L taobao-components:V-flash #PWR?
-U 1 1 5C2679A3
-P 11150 5600
-F 0 "#PWR?" H 11150 5450 50  0001 C CNN
-F 1 "V-flash" H 11200 5750 50  0000 C CNN
-F 2 "" H 11150 5600 50  0001 C CNN
-F 3 "" H 11150 5600 50  0001 C CNN
-	1    11150 5600
-	1    0    0    -1
-$EndComp
-$Comp
 L taobao-c:C105,0603 C?
 U 1 1 5C267ABC
@@
 	11300 6100 11150 6100
 Connection ~ 11150 6100
-$Comp
-L taobao-components:V-flash #PWR?
-U 1 1 5C26DB4B
-P 12250 5650
-F 0 "#PWR?" H 12250 5500 50  0001 C CNN
-F 1 "V-flash" H 12300 5800 50  0000 C CNN
-F 2 "" H 12250 5650 50  0001 C CNN
-F 3 "" H 12250 5650 50  0001 C CNN
-	1    12250 5650
-	1    0    0    -1
-$EndComp
 $Comp
 L taobao-r:R103,0603 R?
@@
 	13700 5850 12750 5850
 $Comp
-L taobao-components:V-flash #PWR?
-U 1 1 5C5BE76C
-P 5650 2100
-F 0 "#PWR?" H 5650 1950 50  0001 C CNN
-F 1 "V-flash" H 5700 2250 50  0000 C CNN
-F 2 "" H 5650 2100 50  0001 C CNN
-F 3 "" H 5650 2100 50  0001 C CNN
-	1    5650 2100
-	1    0    0    -1
-$EndComp
-$Comp
 L taobao-r:R0,0603 R?
 U 1 1 5C5C07D8
@@
 	1    0    0    -1
 $EndComp
+$Comp
+L taobao-components:VCC-FLASH #PWR?
+U 1 1 5C4011A8
+P 5650 2100
+F 0 "#PWR?" H 5650 1950 50  0001 C CNN
+F 1 "VCC-FLASH" H 5700 2250 50  0000 C CNN
+F 2 "" H 5650 2100 50  0001 C CNN
+F 3 "" H 5650 2100 50  0001 C CNN
+	1    5650 2100
+	1    0    0    -1
+$EndComp
+$Comp
+L taobao-components:VCC-FLASH #PWR?
+U 1 1 5C401637
+P 12400 2050
+F 0 "#PWR?" H 12400 1900 50  0001 C CNN
+F 1 "VCC-FLASH" H 12450 2200 50  0000 C CNN
+F 2 "" H 12400 2050 50  0001 C CNN
+F 3 "" H 12400 2050 50  0001 C CNN
+	1    12400 2050
+	1    0    0    -1
+$EndComp
+$Comp
+L taobao-components:VCC-FLASH #PWR?
+U 1 1 5C4016FB
+P 11150 5600
+F 0 "#PWR?" H 11150 5450 50  0001 C CNN
+F 1 "VCC-FLASH" H 11200 5750 50  0000 C CNN
+F 2 "" H 11150 5600 50  0001 C CNN
+F 3 "" H 11150 5600 50  0001 C CNN
+	1    11150 5600
+	1    0    0    -1
+$EndComp
+$Comp
+L taobao-components:VCC-FLASH #PWR?
+U 1 1 5C4018A0
+P 12250 5650
+F 0 "#PWR?" H 12250 5500 50  0001 C CNN
+F 1 "VCC-FLASH" H 12300 5800 50  0000 C CNN
+F 2 "" H 12250 5650 50  0001 C CNN
+F 3 "" H 12250 5650 50  0001 C CNN
+	1    12250 5650
+	1    0    0    -1
+$EndComp
