File: CPU_DECOUPLE_CAP.sch (KiCad schematic (older format))
At the start: 12 parts

Commit message: update power mark,
Connections:
- net labels added: VCC-IO
- net labels removed: Vcc-io
Changed lines of the file:
@@
 $Descr A3 16535 11693
 encoding utf-8
-Sheet 33 33
+Sheet 33 34
 Title ""
 Date ""
@@
 $EndBitmap
 $Comp
-L taobao-components:Vcc-io #PWR?
-U 1 1 5C7AFC79
-P 6950 2900
-F 0 "#PWR?" H 6950 2750 50  0001 C CNN
-F 1 "Vcc-io" H 7000 3050 50  0000 C CNN
-F 2 "" H 6950 2900 50  0001 C CNN
-F 3 "" H 6950 2900 50  0001 C CNN
-	1    6950 2900
-	1    0    0    -1
-$EndComp
-$Comp
 L taobao-c:C105,0603 C?
 U 1 1 5C7AFCFD
 P 6950 3150
+AR Path="/5C273FE9/5C7AC496/5C7AFCFD" Ref="C?"  Part="1"
+AR Path="/5C7B767A/5C7AC496/5C7AFCFD" Ref="C?"  Part="1"
 F 0 "C?" H 7050 3200 50  0000 L CNN
 F 1 "C105,0603" H 7050 3150 50  0000 L CNN
@@
 U 1 1 5C7AFE33
 P 7300 3150
+AR Path="/5C273FE9/5C7AC496/5C7AFE33" Ref="C?"  Part="1"
+AR Path="/5C7B767A/5C7AC496/5C7AFE33" Ref="C?"  Part="1"
 F 0 "C?" H 7400 3200 50  0000 L CNN
 F 1 "C104,0603" H 7400 3150 50  0000 L CNN
@@
 U 1 1 5C7AFEBF
 P 6950 3500
+AR Path="/5C273FE9/5C7AC496/5C7AFEBF" Ref="#PWR?"  Part="1"
+AR Path="/5C7B767A/5C7AC496/5C7AFEBF" Ref="#PWR?"  Part="1"
 F 0 "#PWR?" H 6950 3250 50  0001 C CNN
 F 1 "GND" H 7000 3300 50  0000 C CNN
@@
 U 1 1 5C7AFF9B
 P 8050 2900
+AR Path="/5C273FE9/5C7AC496/5C7AFF9B" Ref="#PWR?"  Part="1"
+AR Path="/5C7B767A/5C7AC496/5C7AFF9B" Ref="#PWR?"  Part="1"
 F 0 "#PWR?" H 8050 2750 50  0001 C CNN
 F 1 "VDD-CPUX" H 8100 3050 50  0000 C CNN
@@
 U 1 1 5C7B003A
 P 8050 3150
+AR Path="/5C273FE9/5C7AC496/5C7B003A" Ref="C?"  Part="1"
+AR Path="/5C7B767A/5C7AC496/5C7B003A" Ref="C?"  Part="1"
 F 0 "C?" H 8150 3200 50  0000 L CNN
 F 1 "C106,0603" H 8150 3150 50  0000 L CNN
@@
 U 1 1 5C7B008A
 P 8350 3150
+AR Path="/5C273FE9/5C7AC496/5C7B008A" Ref="C?"  Part="1"
+AR Path="/5C7B767A/5C7AC496/5C7B008A" Ref="C?"  Part="1"
 F 0 "C?" H 8450 3200 50  0000 L CNN
 F 1 "C105,0603" H 8450 3150 50  0000 L CNN
@@
 U 1 1 5C7B00E6
 P 8600 3150
+AR Path="/5C273FE9/5C7AC496/5C7B00E6" Ref="C?"  Part="1"
+AR Path="/5C7B767A/5C7AC496/5C7B00E6" Ref="C?"  Part="1"
 F 0 "C?" H 8700 3200 50  0000 L CNN
 F 1 "C105,0603" H 8700 3150 50  0000 L CNN
@@
 U 1 1 5C7B012A
 P 8850 3150
+AR Path="/5C273FE9/5C7AC496/5C7B012A" Ref="C?"  Part="1"
+AR Path="/5C7B767A/5C7AC496/5C7B012A" Ref="C?"  Part="1"
 F 0 "C?" H 8950 3200 50  0000 L CNN
 F 1 "C104,0603" H 8950 3150 50  0000 L CNN
@@
 U 1 1 5C7B0176
 P 9100 3150
+AR Path="/5C273FE9/5C7AC496/5C7B0176" Ref="C?"  Part="1"
+AR Path="/5C7B767A/5C7AC496/5C7B0176" Ref="C?"  Part="1"
 F 0 "C?" H 9200 3200 50  0000 L CNN
 F 1 "C104,0603" H 9200 3150 50  0000 L CNN
@@
 U 1 1 5C7B04C3
 P 8050 3500
+AR Path="/5C273FE9/5C7AC496/5C7B04C3" Ref="#PWR?"  Part="1"
+AR Path="/5C7B767A/5C7AC496/5C7B04C3" Ref="#PWR?"  Part="1"
 F 0 "#PWR?" H 8050 3250 50  0001 C CNN
 F 1 "GND" H 8100 3300 50  0000 C CNN
@@
 U 1 1 5C7B3F78
 P 9750 2900
+AR Path="/5C273FE9/5C7AC496/5C7B3F78" Ref="#PWR?"  Part="1"
+AR Path="/5C7B767A/5C7AC496/5C7B3F78" Ref="#PWR?"  Part="1"
 F 0 "#PWR?" H 9750 2750 50  0001 C CNN
 F 1 "Vdd-1V2-sys" H 9800 3050 50  0000 C CNN
@@
 U 1 1 5C7B40A6
 P 9750 3150
+AR Path="/5C273FE9/5C7AC496/5C7B40A6" Ref="C?"  Part="1"
+AR Path="/5C7B767A/5C7AC496/5C7B40A6" Ref="C?"  Part="1"
 F 0 "C?" H 9850 3200 50  0000 L CNN
 F 1 "C106,0603" H 9850 3150 50  0000 L CNN
@@
 U 1 1 5C7B40AC
 P 10050 3150
+AR Path="/5C273FE9/5C7AC496/5C7B40AC" Ref="C?"  Part="1"
+AR Path="/5C7B767A/5C7AC496/5C7B40AC" Ref="C?"  Part="1"
 F 0 "C?" H 10150 3200 50  0000 L CNN
 F 1 "C105,0603" H 10150 3150 50  0000 L CNN
@@
 U 1 1 5C7B40B2
 P 10300 3150
+AR Path="/5C273FE9/5C7AC496/5C7B40B2" Ref="C?"  Part="1"
+AR Path="/5C7B767A/5C7AC496/5C7B40B2" Ref="C?"  Part="1"
 F 0 "C?" H 10400 3200 50  0000 L CNN
 F 1 "C105,0603" H 10400 3150 50  0000 L CNN
@@
 U 1 1 5C7B40B8
 P 10550 3150
+AR Path="/5C273FE9/5C7AC496/5C7B40B8" Ref="C?"  Part="1"
+AR Path="/5C7B767A/5C7AC496/5C7B40B8" Ref="C?"  Part="1"
 F 0 "C?" H 10650 3200 50  0000 L CNN
 F 1 "C104,0603" H 10650 3150 50  0000 L CNN
@@
 U 1 1 5C7B40BE
 P 10800 3150
+AR Path="/5C273FE9/5C7AC496/5C7B40BE" Ref="C?"  Part="1"
+AR Path="/5C7B767A/5C7AC496/5C7B40BE" Ref="C?"  Part="1"
 F 0 "C?" H 10900 3200 50  0000 L CNN
 F 1 "C104,0603" H 10900 3150 50  0000 L CNN
@@
 U 1 1 5C7B40D2
 P 9750 3500
+AR Path="/5C273FE9/5C7AC496/5C7B40D2" Ref="#PWR?"  Part="1"
+AR Path="/5C7B767A/5C7AC496/5C7B40D2" Ref="#PWR?"  Part="1"
 F 0 "#PWR?" H 9750 3250 50  0001 C CNN
 F 1 "GND" H 9800 3300 50  0000 C CNN
@@
 	10800 3400 10550 3400
 Connection ~ 10550 3400
+$Comp
+L taobao-components:VCC-IO #PWR?
+U 1 1 5C7D8921
+P 6950 2900
+F 0 "#PWR?" H 6950 2750 50  0001 C CNN
+F 1 "VCC-IO" H 7000 3050 50  0000 C CNN
+F 2 "" H 6950 2900 50  0001 C CNN
+F 3 "" H 6950 2900 50  0001 C CNN
+	1    6950 2900
+	1    0    0    -1
+$EndComp
 $EndSCHEMATC
