File: allwinner-H3-tryout.sch (KiCad schematic (older format))
At the start: 4 parts

Commit message: update power mark,
Changed lines of the file:
@@
 $Descr A4 11693 8268
 encoding utf-8
-Sheet 1 33
+Sheet 1 34
 Title ""
 Date ""
@@
 F1 "H3_CPU.sch" 50
 $EndSheet
+$Sheet
+S 700  2150 1050 900
+U 5C7B767A
+F0 "power_rail" 50
+F1 "power_rail.sch" 50
+$EndSheet
 $EndSCHEMATC
