File: cpus.sch (KiCad schematic (older format))
At the start: 7 parts

Commit message: update power mark,
Connections:
- net labels added: VCC-IO
- net labels removed: Vcc-io
Changed lines of the file:
@@
 $Descr A3 16535 11693
 encoding utf-8
-Sheet 18 33
+Sheet 18 34
 Title ""
 Date ""
@@
 AR Path="/5C273FE9/5C29102D/5C66DCD6" Ref="U?"  Part="10"
 AR Path="/5C273FE9/5C786D7F/5C66DCD6" Ref="U?"  Part="10"
+AR Path="/5C7B767A/5C29102D/5C66DCD6" Ref="U?"  Part="10"
 F 0 "U?" H 8800 6500 50  0000 C CNN
 F 1 "allwinner-H3" H 8800 6400 50  0000 C CNN
@@
 AR Path="/5C273FE9/5C29102D/5C66DDB7" Ref="R?"  Part="1"
 AR Path="/5C273FE9/5C786D7F/5C66DDB7" Ref="R?"  Part="1"
+AR Path="/5C7B767A/5C29102D/5C66DDB7" Ref="R?"  Part="1"
 F 0 "R?" H 9900 4800 50  0000 L CNN
 F 1 "R103,0603" H 9900 4750 50  0000 L CNN
@@
 AR Path="/5C273FE9/5C29102D/5C66DEE1" Ref="R?"  Part="1"
 AR Path="/5C273FE9/5C786D7F/5C66DEE1" Ref="R?"  Part="1"
+AR Path="/5C7B767A/5C29102D/5C66DEE1" Ref="R?"  Part="1"
 F 0 "R?" H 10150 4800 50  0000 L CNN
 F 1 "R_NC,0603" H 10150 4750 50  0000 L CNN
@@
 AR Path="/5C273FE9/5C29102D/5C66DFE7" Ref="R?"  Part="1"
 AR Path="/5C273FE9/5C786D7F/5C66DFE7" Ref="R?"  Part="1"
+AR Path="/5C7B767A/5C29102D/5C66DFE7" Ref="R?"  Part="1"
 F 0 "R?" H 10400 4800 50  0000 L CNN
 F 1 "R103,0603" H 10400 4750 50  0000 L CNN
@@
 AR Path="/5C273FE9/5C29102D/5C66E0E9" Ref="#PWR?"  Part="1"
 AR Path="/5C273FE9/5C786D7F/5C66E0E9" Ref="#PWR?"  Part="1"
+AR Path="/5C7B767A/5C29102D/5C66E0E9" Ref="#PWR?"  Part="1"
 F 0 "#PWR?" H 9800 4300 50  0001 C CNN
 F 1 "GND" H 9800 4350 50  0000 C CNN
@@
 Wire Wire Line
 	9800 4550 9800 4650
-$Comp
-L taobao-components:Vcc-io #PWR?
-U 1 1 5C66E1C8
-P 10050 4550
-AR Path="/5C66D9B1/5C66E1C8" Ref="#PWR?"  Part="1"
-AR Path="/5C2567C9/5C66E1C8" Ref="#PWR?"  Part="1"
-AR Path="/5C273FE9/5C29102D/5C66E1C8" Ref="#PWR?"  Part="1"
-AR Path="/5C273FE9/5C786D7F/5C66E1C8" Ref="#PWR?"  Part="1"
-F 0 "#PWR?" H 10050 4400 50  0001 C CNN
-F 1 "Vcc-io" H 10100 4700 50  0000 C CNN
-F 2 "" H 10050 4550 50  0001 C CNN
-F 3 "" H 10050 4550 50  0001 C CNN
-	1    10050 4550
-	1    0    0    -1
-$EndComp
 Wire Wire Line
 	10050 4550 10050 4650
@@
 AR Path="/5C273FE9/5C29102D/5C671FBA" Ref="#PWR?"  Part="1"
 AR Path="/5C273FE9/5C786D7F/5C671FBA" Ref="#PWR?"  Part="1"
+AR Path="/5C7B767A/5C29102D/5C671FBA" Ref="#PWR?"  Part="1"
 F 0 "#PWR?" H 10300 4400 50  0001 C CNN
 F 1 "VCC-RTC" H 10350 4700 50  0000 C CNN
@@
 	9600 6100 10600 6100
 $Comp
-L taobao-components:Vcc-io #PWR?
-U 1 1 5C251BB7
-P 8550 7100
-AR Path="/5C66D9B1/5C251BB7" Ref="#PWR?"  Part="1"
-AR Path="/5C2567C9/5C251BB7" Ref="#PWR?"  Part="1"
-AR Path="/5C273FE9/5C29102D/5C251BB7" Ref="#PWR?"  Part="1"
-AR Path="/5C273FE9/5C786D7F/5C251BB7" Ref="#PWR?"  Part="1"
-F 0 "#PWR?" H 8550 6950 50  0001 C CNN
-F 1 "Vcc-io" H 8600 7250 50  0000 C CNN
-F 2 "" H 8550 7100 50  0001 C CNN
-F 3 "" H 8550 7100 50  0001 C CNN
-	1    8550 7100
-	1    0    0    -1
-$EndComp
-$Comp
 L taobao-components:R_NC,0402 R?
 U 1 1 5C251CA2
@@
 AR Path="/5C273FE9/5C29102D/5C251CA2" Ref="R?"  Part="1"
 AR Path="/5C273FE9/5C786D7F/5C251CA2" Ref="R?"  Part="1"
+AR Path="/5C7B767A/5C29102D/5C251CA2" Ref="R?"  Part="1"
 F 0 "R?" H 8650 7450 50  0000 L CNN
 F 1 "R_NC,0402" H 8650 7400 50  0000 L CNN
@@
 AR Path="/5C273FE9/5C29102D/5C253FFD" Ref="#PWR?"  Part="1"
 AR Path="/5C273FE9/5C786D7F/5C253FFD" Ref="#PWR?"  Part="1"
+AR Path="/5C7B767A/5C29102D/5C253FFD" Ref="#PWR?"  Part="1"
 F 0 "#PWR?" H 10150 6950 50  0001 C CNN
 F 1 "VCC-RTC" H 10200 7250 50  0000 C CNN
@@
 AR Path="/5C273FE9/5C29102D/5C2540EB" Ref="R?"  Part="1"
 AR Path="/5C273FE9/5C786D7F/5C2540EB" Ref="R?"  Part="1"
+AR Path="/5C7B767A/5C29102D/5C2540EB" Ref="R?"  Part="1"
 F 0 "R?" H 10250 7400 50  0000 L CNN
 F 1 "R103,0603" H 10250 7350 50  0000 L CNN
@@
 AR Path="/5C273FE9/5C29102D/5C254238" Ref="R?"  Part="1"
 AR Path="/5C273FE9/5C786D7F/5C254238" Ref="R?"  Part="1"
+AR Path="/5C7B767A/5C29102D/5C254238" Ref="R?"  Part="1"
 F 0 "R?" H 10600 7400 50  0000 L CNN
 F 1 "R103,0603" H 10600 7350 50  0000 L CNN
@@
 EndData
 $EndBitmap
+$Comp
+L taobao-components:VCC-IO #PWR?
+U 1 1 5C7D8841
+P 10050 4550
+F 0 "#PWR?" H 10050 4400 50  0001 C CNN
+F 1 "VCC-IO" H 10100 4700 50  0000 C CNN
+F 2 "" H 10050 4550 50  0001 C CNN
+F 3 "" H 10050 4550 50  0001 C CNN
+	1    10050 4550
+	1    0    0    -1
+$EndComp
+$Comp
+L taobao-components:VCC-IO #PWR?
+U 1 1 5C7D887F
+P 8550 7100
+F 0 "#PWR?" H 8550 6950 50  0001 C CNN
+F 1 "VCC-IO" H 8600 7250 50  0000 C CNN
+F 2 "" H 8550 7100 50  0001 C CNN
+F 3 "" H 8550 7100 50  0001 C CNN
+	1    8550 7100
+	1    0    0    -1
+$EndComp
 $EndSCHEMATC
