File: CPU_SYS.sch (KiCad schematic (older format))
At the start: 11 parts

Commit message: update,
Changed lines of the file:
@@
 	7100 4700 6600 4700
 Connection ~ 6600 4700
-$Comp
-L taobao-components:VCC3V3-PLL #PWR?
-U 1 1 5C2BBF0E
-P 10300 4900
-AR Path="/5C273FE9/5C2B8F59/5C2BBF0E" Ref="#PWR?"  Part="1"
-AR Path="/5C273FE9/5C2D084A/5C2BBF0E" Ref="#PWR?"  Part="1"
-AR Path="/5C7B767A/5C2B8F59/5C2BBF0E" Ref="#PWR?"  Part="1"
-F 0 "#PWR?" H 10300 4750 50  0001 C CNN
-F 1 "VCC3V3-PLL" H 10350 5050 50  0000 C CNN
-F 2 "" H 10300 4900 50  0001 C CNN
-F 3 "" H 10300 4900 50  0001 C CNN
-	1    10300 4900
-	1    0    0    -1
-$EndComp
 Text GLabel 9900 4050 2    50   Input ~ 0
 X32K-WIFI
