File: RTC.sch (KiCad schematic (older format))
At the start: 11 parts

Commit message: update power mark,
Connections:
- net labels added: VCC-5V, VCC-IO
- net labels removed: Vcc-5V, Vcc-io
Changed lines of the file:
@@
 $Descr A4 11693 8268
 encoding utf-8
-Sheet 9 33
+Sheet 9 34
 Title ""
 Date ""
@@
 $EndBitmap
 $Comp
-L taobao-components:Vcc-io #PWR?
-U 1 1 5C21CF1E
-P 4400 4300
-F 0 "#PWR?" H 4400 4150 50  0001 C CNN
-F 1 "Vcc-io" H 4405 4423 50  0000 C CNN
-F 2 "" H 4400 4300 50  0001 C CNN
-F 3 "" H 4400 4300 50  0001 C CNN
-	1    4400 4300
-	1    0    0    -1
-$EndComp
-$Comp
 L taobao-led:LED_GREEN,0603 D?
 U 1 1 5C21D0E8
@@
 $EndComp
 $Comp
-L taobao-components:Vcc-io #PWR?
-U 1 1 5C21D451
-P 3600 4800
-F 0 "#PWR?" H 3600 4650 50  0001 C CNN
-F 1 "Vcc-io" H 3605 4923 50  0000 C CNN
-F 2 "" H 3600 4800 50  0001 C CNN
-F 3 "" H 3600 4800 50  0001 C CNN
-	1    3600 4800
-	1    0    0    -1
-$EndComp
-$Comp
 L taobao-r:R103,0603 R?
 U 1 1 5C21D52C
@@
 $EndComp
 $Comp
-L taobao-components:Vcc-io #PWR?
-U 1 1 5C226D11
-P 7400 3750
-F 0 "#PWR?" H 7400 3600 50  0001 C CNN
-F 1 "Vcc-io" H 7405 3873 50  0000 C CNN
-F 2 "" H 7400 3750 50  0001 C CNN
-F 3 "" H 7400 3750 50  0001 C CNN
-	1    7400 3750
-	1    0    0    -1
-$EndComp
-$Comp
 L power:GND #PWR?
 U 1 1 5C22705C
@@
 Text GLabel 7100 5850 0    50   Input ~ 0
 SPDIF-OUT
-$Comp
-L taobao-components:Vcc-5V #PWR?
-U 1 1 5C22F514
-P 9500 3750
-F 0 "#PWR?" H 9500 3600 50  0001 C CNN
-F 1 "Vcc-5V" H 9505 3873 50  0000 C CNN
-F 2 "" H 9500 3750 50  0001 C CNN
-F 3 "" H 9500 3750 50  0001 C CNN
-	1    9500 3750
-	1    0    0    -1
-$EndComp
 Wire Wire Line
 	9500 3750 9500 4050
@@
 EndData
 $EndBitmap
+$Comp
+L taobao-components:VCC-IO #PWR?
+U 1 1 5C7D7D06
+P 4400 4300
+F 0 "#PWR?" H 4400 4150 50  0001 C CNN
+F 1 "VCC-IO" H 4450 4450 50  0000 C CNN
+F 2 "" H 4400 4300 50  0001 C CNN
+F 3 "" H 4400 4300 50  0001 C CNN
+	1    4400 4300
+	1    0    0    -1
+$EndComp
+$Comp
+L taobao-components:VCC-IO #PWR?
+U 1 1 5C7D7D2E
+P 3600 4800
+F 0 "#PWR?" H 3600 4650 50  0001 C CNN
+F 1 "VCC-IO" H 3650 4950 50  0000 C CNN
+F 2 "" H 3600 4800 50  0001 C CNN
+F 3 "" H 3600 4800 50  0001 C CNN
+	1    3600 4800
+	1    0    0    -1
+$EndComp
+$Comp
+L taobao-components:VCC-IO #PWR?
+U 1 1 5C7D7F5F
+P 7400 3750
+F 0 "#PWR?" H 7400 3600 50  0001 C CNN
+F 1 "VCC-IO" H 7450 3900 50  0000 C CNN
+F 2 "" H 7400 3750 50  0001 C CNN
+F 3 "" H 7400 3750 50  0001 C CNN
+	1    7400 3750
+	1    0    0    -1
+$EndComp
+$Comp
+L taobao-components:VCC-5V #PWR?
+U 1 1 5C7DB90F
+P 9500 3750
+F 0 "#PWR?" H 9500 3600 50  0001 C CNN
+F 1 "VCC-5V" H 9550 3900 50  0000 C CNN
+F 2 "" H 9500 3750 50  0001 C CNN
+F 3 "" H 9500 3750 50  0001 C CNN
+	1    9500 3750
+	1    0    0    -1
+$EndComp
 $EndSCHEMATC
